File: placa-principal-angra/placa-principal-angra.kicad_pcb (KiCad board)
At the start: 2 copper layers, 23 parts, among them J1 ENTRADA-PH, J10 SONAR-4, J11 SONAR-5, J12 MPU, J2 SAÍDA PH, J7 SONAR-1, J8 SONAR-2, J9 SONAR-3, U1 ESP32-S3-DevKitC

Commit message: feat: Trazendo os componentes pra placa
Parts:
- moved J1 164.6 mm to (113.8, 130.2)
- moved J10 164.6 mm to (127.8, 114.0)
- moved J11 164.6 mm to (132.3, 114.0)
- moved J2 164.6 mm to (117.3, 130.2)
- moved J3 164.6 mm to (113.8, 125.7)
- moved J4 164.6 mm to (117.3, 125.7)
- moved J5 164.6 mm to (120.9, 125.7)
- moved J6 164.6 mm to (124.4, 125.7)
- moved J7 164.6 mm to (114.0, 114.0)
- moved J8 164.6 mm to (118.6, 114.0)
- moved J9 164.6 mm to (123.2, 114.0)
- moved R1 164.6 mm to (113.7, 73.2)
- moved R10 164.6 mm to (113.7, 109.7)
- moved R2 164.6 mm to (113.7, 77.2)
- moved R3 164.6 mm to (113.7, 81.3)
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