File: placa-principal-angra/placa-principal-angra.kicad_sch (KiCad schematic)
At the start: 0 parts

Commit message: feat: salvei
Parts:
- added J1: ENTRADA-PH, Connector_PinSocket_1.00mm:PinSocket_1x08_P1.00mm_Vertical, symbol Connector_Generic:Conn_01x08
- added J10: SONAR-4, Connector_PinSocket_2.54mm:PinSocket_1x04_P2.54mm_Vertical, symbol Connector_Generic:Conn_01x04
- added J11: SONAR-5, Connector_PinSocket_2.54mm:PinSocket_1x04_P2.54mm_Vertical, symbol Connector_Generic:Conn_01x04
- added J12: MPU, Connector_PinSocket_2.54mm:PinSocket_1x04_P2.54mm_Vertical, symbol Connector_Generic:Conn_01x04
- added J2: SAÍDA PH, Connector_PinSocket_1.00mm:PinSocket_1x08_P1.00mm_Vertical, symbol Connector_Generic:Conn_01x08
- added J3, J4, J5, J6: (no value), Connector_PinSocket_1.00mm:PinSocket_1x02_P1.00mm_Vertical, symbol Connector_Generic:Conn_01x02
- added J7: SONAR-1, Connector_PinSocket_2.54mm:PinSocket_1x04_P2.54mm_Vertical, symbol Connector_Generic:Conn_01x04
- added J8: SONAR-2, Connector_PinSocket_2.54mm:PinSocket_1x04_P2.54mm_Vertical, symbol Connector_Generic:Conn_01x04
- added J9: SONAR-3, Connector_PinSocket_2.54mm:PinSocket_1x04_P2.54mm_Vertical, symbol Connector_Generic:Conn_01x04
- added R1, R3, R5, R7, R9: 1K, Resistor_THT:R_Axial_DIN0207_L6.3mm_D2.5mm_P5.08mm_Vertical, symbol Device:R_Small
- added R10, R2, R4, R6, R8: 2K, Resistor_THT:R_Axial_DIN0207_L6.3mm_D2.5mm_P5.08mm_Vertical, symbol Device:R_Small
- added U1: ESP32-S3-DevKitC, PCM_Espressif:ESP32-S3-DevKitC, symbol PCM_Espressif:ESP32-S3-DevKitC
Connections:
- new net: J11.2 (Pin_2), R9.1
- new net: J9.2 (Pin_2), R5.1
- new net: J10.2 (Pin_2), R7.1
- new net: J8.2 (Pin_2), R3.1
- new net: J7.2 (Pin_2), R1.1
- new net: U1.22 (GND), U1.23 (GND), U1.24 (GND), U1.44 (GND)
- new net 3V3: J12.4 (Pin_4), J2.7 (Pin_7), U1.1 (3V3), U1.2 (3V3)
- new net 5V: J10.4 (Pin_4), J11.4 (Pin_4), J7.4 (Pin_4), J8.4 (Pin_4), J9.4 (Pin_4), U1.21 (5V)
- new net A01: J2.5 (Pin_5), J5.1 (Pin_1), J6.2 (Pin_2)
- new net A02: J2.4 (Pin_4), J5.2 (Pin_2), J6.1 (Pin_1)
- new net B01: J2.2 (Pin_2), J3.1 (Pin_1), J4.2 (Pin_2)
- new net B02: J2.3 (Pin_3), J3.2 (Pin_2), J4.1 (Pin_1)
- new net ECHO1: R1.2, R2.2, U1.17 (GPIO11/ADC2_CH0)
- new net ECHO2: R3.2, R4.2, U1.19 (GPIO13/ADC2_CH2)
- new net ECHO3: R5.2, R6.2, U1.27 (GPIO21)
- new net ECHO4: R7.2, R8.2, U1.33 (GPIO36)
- new net ECHO5: R10.2, R9.2, U1.35 (GPIO38)
- new net GND: J1.8 (Pin_8), J10.1 (Pin_1), J11.1 (Pin_1), J12.3 (Pin_3), J2.1 (Pin_1), J2.6 (Pin_6), J7.1 (Pin_1), J8.1 (Pin_1), J9.1 (Pin_1), R10.1, R2.1, R4.1, R6.1, R8.1
- new net GPIO15: J1.7 (Pin_7), U1.8 (GPIO15/ADC2_CH4/32K_P)
- new net GPIO16: J1.5 (Pin_5), U1.9 (GPIO16/ADC2_CH5/32K_N)
- new net GPIO17: J1.6 (Pin_6), U1.10 (GPIO17/ADC2_CH6)
- new net GPIO4: J1.4 (Pin_4), U1.4 (GPIO4/ADC1_CH3)
- new net GPIO5: J1.1 (Pin_1), U1.5 (GPIO5/ADC1_CH4)
- new net GPIO6: J1.3 (Pin_3), U1.6 (GPIO6/ADC1_CH5)
- new net GPIO7: J1.2 (Pin_2), U1.7 (GPIO7/ADC1_CH6)
- new net SCL: J12.1 (Pin_1), U1.15 (GPIO9/ADC1_CH8)
- new net SDA: J12.2 (Pin_2), U1.12 (GPIO8/ADC1_CH7)
- new net TRIG1: J7.3 (Pin_3), U1.16 (GPIO10/ADC1_CH9)
- new net TRIG2: J8.3 (Pin_3), U1.18 (GPIO12/ADC2_CH1)
- new net TRIG3: J9.3 (Pin_3), U1.11 (GPIO18/ADC2_CH7)
- new net TRIG4: J10.3 (Pin_3), U1.32 (GPIO35)
- new net TRIG5: J11.3 (Pin_3), U1.34 (GPIO37)
- new net VM: J2.8 (Pin_8)
- no-connect marks 0 -> 18
