File: placa-principal-angra/_restore_backup_2026-06-26T15-26-39-179/placa-principal-angra.kicad_pcb (KiCad board)
At the start: 2 copper layers, 28 parts, among them J1 ENTRADA-PH, J10 SONAR-4, J11 SONAR-5, J12 MPU, J2 SAÍDA PH, J7 SONAR-1, J8 SONAR-2, J9 SONAR-3, U1 ESP32-S3-DevKitC

Commit message: feat: Ajustando o roteamento
Parts:
- removed R11, R12, R13, R14, R15: 1K, Resistor_THT:R_Axial_DIN0207_L6.3mm_D2.5mm_P5.08mm_Vertical
- R10, R2, R4, R6, R8: value 1K -> 2K
- moved R10 123.8 mm to (32.5, 113.8), turned to 0 degrees
- moved R6 121.9 mm to (32.5, 97.6), turned to 0 degrees
- moved R5 121.9 mm to (32.5, 93.5), turned to 0 degrees
- moved R9 109.8 mm to (32.5, 109.8), turned to 0 degrees
- moved R8 109.7 mm to (32.5, 105.7), turned to 0 degrees
- moved R7 109.6 mm to (32.5, 101.7), turned to 0 degrees
- moved J6 74.5 mm to (43.2, 129.8)
- moved J3 74.5 mm to (32.5, 129.8)
- moved J4 74.5 mm to (36.1, 129.8)
- moved J5 74.5 mm to (39.6, 129.8)
- moved R3 40.9 mm to (134.5, 94.5)
- moved J11 38.6 mm to (143.0, 129.2), turned to 0 degrees
- moved R4 36.7 mm to (135.8, 87.5)
- moved J7 34.2 mm to (143.0, 71.5), turned to 0 degrees
- moved U1 32.3 mm to (67.9, 58.4)
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Connections:
- R10 pad 1: Net-(J10-Pin_2) -> /GND
- R10 pad 2: /ECHO4 -> /ECHO5
- R2 pad 1: Net-(R2-Pad1) -> /GND
- R3 pad 1: /GND -> Net-(J8-Pin_2)
- R3 pad 2: Net-(R2-Pad1) -> /ECHO2
- R4 pad 1: Net-(J8-Pin_2) -> /GND
- R5 pad 1: Net-(R5-Pad1) -> Net-(J9-Pin_2)
- R5 pad 2: /ECHO2 -> /ECHO3
- R6 pad 2: Net-(R5-Pad1) -> /ECHO3
- R7 pad 1: Net-(J9-Pin_2) -> Net-(J10-Pin_2)
- R7 pad 2: /ECHO3 -> /ECHO4
- R8 pad 1: Net-(R8-Pad1) -> /GND
- R8 pad 2: /ECHO3 -> /ECHO4
- R9 pad 1: /GND -> Net-(J11-Pin_2)
- R9 pad 2: Net-(R8-Pad1) -> /ECHO5
