File: placa-principal-angra/_restore_backup_2026-06-26T15-26-39-179/placa-principal-angra.kicad_sch (KiCad schematic)
At the start: 28 parts, among them J1 ENTRADA-PH, J10 SONAR-4, J11 SONAR-5, J12 MPU, J2 SAÍDA PH, J7 SONAR-1, J8 SONAR-2, J9 SONAR-3, U1 ESP32-S3-DevKitC

Commit message: feat: Ajustando o roteamento
Parts:
- J10: value SONAR-4 -> SONAR-1
- J11: value SONAR-5 -> SONAR-1
- J8: value SONAR-2 -> SONAR-1
- J9: value SONAR-3 -> SONAR-1
Changed lines of the file:
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@@
 			)
 		)
-		(property "Value" "SONAR-3"
+		(property "Value" "SONAR-1"
 			(at 214.63 107.95 0)
 			(show_name no)
@@
 			)
 		)
-		(property "Value" "SONAR-4"
+		(property "Value" "SONAR-1"
 			(at 182.88 133.35 0)
 			(show_name no)
@@
 			)
 		)
-		(property "Value" "SONAR-5"
+		(property "Value" "SONAR-1"
 			(at 213.36 134.62 0)
 			(show_name no)
@@
 			)
 		)
-		(property "Value" "SONAR-2"
+		(property "Value" "SONAR-1"
 			(at 187.96 107.95 0)
 			(show_name no)
